Commit message: Rename openarm_grip to openarm

File: openarm_description/urdf/materials.xacro (robot description, xacro)
@@ -1,4 +1,4 @@
 <?xml version="1.0" ?>
-<robot name="openarm_grip" xmlns:xacro="http://www.ros.org/wiki/xacro" >
+<robot name="openarm" xmlns:xacro="http://www.ros.org/wiki/xacro" >
 <material name="silver">
   <color rgba="0.700 0.700 0.700 1.000"/>

File: openarm_description/urdf/openarm_grip.urdf (robot description, URDF)
Before this commit: robot openarm_grip, 11 links, 9 joints
Links:
- link J2_v1_1: geometry collision mesh filename=package://openarm_description/meshes/J2_v1_1.stl scale=0.001 0.001 0.001; visual mesh filename=package://openarm_description/meshes/J2_v1_1.stl scale=0.001 0.001 0.001
- link J3_v1_1: geometry collision mesh filename=package://openarm_description/meshes/J3_v1_1.stl scale=0.001 0.001 0.001; visual mesh filename=package://openarm_description/meshes/J3_v1_1.stl scale=0.001 0.001 0.001
- link J4_v1_1: geometry collision mesh filename=package://openarm_description/meshes/J4_v1_1.stl scale=0.001 0.001 0.001; visual mesh filename=package://openarm_description/meshes/J4_v1_1.stl scale=0.001 0.001 0.001
- link J5_v1_1: geometry collision mesh filename=package://openarm_description/meshes/J5_v1_1.stl scale=0.001 0.001 0.001; visual mesh filename=package://openarm_description/meshes/J5_v1_1.stl scale=0.001 0.001 0.001
- link J6_v1_1: geometry collision mesh filename=package://openarm_description/meshes/J6_v1_1.stl scale=0.001 0.001 0.001; visual mesh filename=package://openarm_description/meshes/J6_v1_1.stl scale=0.001 0.001 0.001
- link J7_v1_1: geometry collision mesh filename=package://openarm_description/meshes/J7_v1_1.stl scale=0.001 0.001 0.001; visual mesh filename=package://openarm_description/meshes/J7_v1_1.stl scale=0.001 0.001 0.001
- link base_link: geometry collision mesh filename=package://openarm_description/meshes/base_link.stl scale=0.001 0.001 0.001; visual mesh filename=package://openarm_description/meshes/base_link.stl scale=0.001 0.001 0.001
- link grip_attach_1: geometry collision mesh filename=package://openarm_description/meshes/grip_attach_1.stl scale=0.001 0.001 0.001; visual mesh filename=package://openarm_description/meshes/grip_attach_1.stl scale=0.001 0.001 0.001
- link left_jaw_1: geometry collision mesh filename=package://openarm_description/meshes/left_jaw_1.stl scale=0.001 0.001 0.001; visual mesh filename=package://openarm_description/meshes/left_jaw_1.stl scale=0.001 0.001 0.001
- link right_jaw_1: geometry collision mesh filename=package://openarm_description/meshes/right_jaw_1.stl scale=0.001 0.001 0.001; visual mesh filename=package://openarm_description/meshes/right_jaw_1.stl scale=0.001 0.001 0.001

File: openarm_description/urdf/openarm_grip.xacro (robot description, xacro)
@@ -1,7 +1,7 @@
 <?xml version="1.0" ?>
-<robot name="openarm_grip" xmlns:xacro="http://www.ros.org/wiki/xacro">
-<xacro:include filename="$(find openarm_grip_description)/urdf/materials.xacro" />
-<xacro:include filename="$(find openarm_grip_description)/urdf/openarm_grip.trans" />
-<xacro:include filename="$(find openarm_grip_description)/urdf/openarm_grip.gazebo" />
+<robot name="openarm" xmlns:xacro="http://www.ros.org/wiki/xacro">
+<xacro:include filename="$(find openarm_description)/urdf/materials.xacro" />
+<xacro:include filename="$(find openarm_description)/urdf/openarm.trans" />
+<xacro:include filename="$(find openarm_description)/urdf/openarm.gazebo" />
 <link name="dummy"/>
 <joint name="dummy_joint" type="fixed">
@@ -19,5 +19,5 @@
     <origin xyz="0 0 0" rpy="0 0 0"/>
     <geometry>
-      <mesh filename="package://openarm_grip_description/meshes/base_link.stl" scale="0.001 0.001 0.001"/>
+      <mesh filename="package://openarm_description/meshes/base_link.stl" scale="0.001 0.001 0.001"/>
     </geometry>
     <material name="silver"/>
@@ -26,5 +26,5 @@
     <origin xyz="0 0 0" rpy="0 0 0"/>
     <geometry>
-      <mesh filename="package://openarm_grip_description/meshes/base_link.stl" scale="0.001 0.001 0.001"/>
+      <mesh filename="package://openarm_description/meshes/base_link.stl" scale="0.001 0.001 0.001"/>
     </geometry>
   </collision>
@@ -39,5 +39,5 @@
     <origin xyz="-0.0 -0.0 0.00225" rpy="0 0 0"/>
     <geometry>
-      <mesh filename="package://openarm_grip_description/meshes/J2_v1_1.stl" scale="0.001 0.001 0.001"/>
+      <mesh filename="package://openarm_description/meshes/J2_v1_1.stl" scale="0.001 0.001 0.001"/>
     </geometry>
     <material name="silver"/>
@@ -46,5 +46,5 @@
     <origin xyz="-0.0 -0.0 0.00225" rpy="0 0 0"/>
     <geometry>
-      <mesh filename="package://openarm_grip_description/meshes/J2_v1_1.stl" scale="0.001 0.001 0.001"/>
+      <mesh filename="package://openarm_description/meshes/J2_v1_1.stl" scale="0.001 0.001 0.001"/>
     </geometry>
   </collision>
@@ -59,5 +59,5 @@
     <origin xyz="-0.02975 0.0 -0.0425" rpy="0 0 0"/>
     <geometry>
-      <mesh filename="package://openarm_grip_description/meshes/J3_v1_1.stl" scale="0.001 0.001 0.001"/>
+      <mesh filename="package://openarm_description/meshes/J3_v1_1.stl" scale="0.001 0.001 0.001"/>
     </geometry>
     <material name="silver"/>
@@ -66,5 +66,5 @@
     <origin xyz="-0.02975 0.0 -0.0425" rpy="0 0 0"/>
     <geometry>
-      <mesh filename="package://openarm_grip_description/meshes/J3_v1_1.stl" scale="0.001 0.001 0.001"/>
+      <mesh filename="package://openarm_description/meshes/J3_v1_1.stl" scale="0.001 0.001 0.001"/>
     </geometry>
   </collision>
@@ -79,5 +79,5 @@
     <origin xyz="0.0 -0.06041 -0.052607" rpy="0 0 0"/>
     <geometry>
-      <mesh filename="package://openarm_grip_description/meshes/J4_v1_1.stl" scale="0.001 0.001 0.001"/>
+      <mesh filename="package://openarm_description/meshes/J4_v1_1.stl" scale="0.001 0.001 0.001"/>
     </geometry>
     <material name="silver"/>
@@ -86,5 +86,5 @@
     <origin xyz="0.0 -0.06041 -0.052607" rpy="0 0 0"/>
     <geometry>
-      <mesh filename="package://openarm_grip_description/meshes/J4_v1_1.stl" scale="0.001 0.001 0.001"/>
+      <mesh filename="package://openarm_description/meshes/J4_v1_1.stl" scale="0.001 0.001 0.001"/>
     </geometry>
   </collision>
@@ -99,5 +99,5 @@
     <origin xyz="-0.029755 -0.298846 -0.0925" rpy="0 0 0"/>
     <geometry>
-      <mesh filename="package://openarm_grip_description/meshes/J5_v1_1.stl" scale="0.001 0.001 0.001"/>
+      <mesh filename="package://openarm_description/meshes/J5_v1_1.stl" scale="0.001 0.001 0.001"/>
     </geometry>
     <material name="silver"/>
@@ -106,5 +106,5 @@
     <origin xyz="-0.029755 -0.298846 -0.0925" rpy="0 0 0"/>
     <geometry>
-      <mesh filename="package://openarm_grip_description/meshes/J5_v1_1.stl" scale="0.001 0.001 0.001"/>
+      <mesh filename="package://openarm_description/meshes/J5_v1_1.stl" scale="0.001 0.001 0.001"/>
     </geometry>
   </collision>
@@ -119,5 +119,5 @@
     <origin xyz="0.0 -0.167496 -0.118765" rpy="0 0 0"/>
     <geometry>
-      <mesh filename="package://openarm_grip_description/meshes/J6_v1_1.stl" scale="0.001 0.001 0.001"/>
+      <mesh filename="package://openarm_description/meshes/J6_v1_1.stl" scale="0.001 0.001 0.001"/>
     </geometry>
     <material name="silver"/>
@@ -126,5 +126,5 @@
     <origin xyz="0.0 -0.167496 -0.118765" rpy="0 0 0"/>
     <geometry>
-      <mesh filename="package://openarm_grip_description/meshes/J6_v1_1.stl" scale="0.001 0.001 0.001"/>
+      <mesh filename="package://openarm_description/meshes/J6_v1_1.stl" scale="0.001 0.001 0.001"/>
     </geometry>
   </collision>
@@ -139,5 +139,5 @@
     <origin xyz="-0.0355 -0.048796 -0.1425" rpy="0 0 0"/>
     <geometry>
-      <mesh filename="package://openarm_grip_description/meshes/J7_v1_1.stl" scale="0.001 0.001 0.001"/>
+      <mesh filename="package://openarm_description/meshes/J7_v1_1.stl" scale="0.001 0.001 0.001"/>
     </geometry>
     <material name="silver"/>
@@ -146,5 +146,5 @@
     <origin xyz="-0.0355 -0.048796 -0.1425" rpy="0 0 0"/>
     <geometry>
-      <mesh filename="package://openarm_grip_description/meshes/J7_v1_1.stl" scale="0.001 0.001 0.001"/>
+      <mesh filename="package://openarm_description/meshes/J7_v1_1.stl" scale="0.001 0.001 0.001"/>
     </geometry>
   </collision>
@@ -159,5 +159,5 @@
     <origin xyz="0.0 -0.051826 -0.15765" rpy="0 0 0"/>
     <geometry>
-      <mesh filename="package://openarm_grip_description/meshes/grip_attach_1.stl" scale="0.001 0.001 0.001"/>
+      <mesh filename="package://openarm_description/meshes/grip_attach_1.stl" scale="0.001 0.001 0.001"/>
     </geometry>
     <material name="silver"/>
@@ -166,5 +166,5 @@
     <origin xyz="0.0 -0.051826 -0.15765" rpy="0 0 0"/>
     <geometry>
-      <mesh filename="package://openarm_grip_description/meshes/grip_attach_1.stl" scale="0.001 0.001 0.001"/>
+      <mesh filename="package://openarm_description/meshes/grip_attach_1.stl" scale="0.001 0.001 0.001"/>
     </geometry>
   </collision>
@@ -179,5 +179,5 @@
     <origin xyz="0.0775 0.069829 -0.169736" rpy="0 0 0"/>
     <geometry>
-      <mesh filename="package://openarm_grip_description/meshes/left_jaw_1.stl" scale="0.001 0.001 0.001"/>
+      <mesh filename="package://openarm_description/meshes/left_jaw_1.stl" scale="0.001 0.001 0.001"/>
     </geometry>
     <material name="silver"/>
@@ -186,5 +186,5 @@
     <origin xyz="0.0775 0.069829 -0.169736" rpy="0 0 0"/>
     <geometry>
-      <mesh filename="package://openarm_grip_description/meshes/left_jaw_1.stl" scale="0.001 0.001 0.001"/>
+      <mesh filename="package://openarm_description/meshes/left_jaw_1.stl" scale="0.001 0.001 0.001"/>
     </geometry>
   </collision>
@@ -199,5 +199,5 @@
     <origin xyz="-0.0775 0.069829 -0.169736" rpy="0 0 0"/>
     <geometry>
-      <mesh filename="package://openarm_grip_description/meshes/right_jaw_1.stl" scale="0.001 0.001 0.001"/>
+      <mesh filename="package://openarm_description/meshes/right_jaw_1.stl" scale="0.001 0.001 0.001"/>
     </geometry>
     <material name="silver"/>
@@ -206,5 +206,5 @@
     <origin xyz="-0.0775 0.069829 -0.169736" rpy="0 0 0"/>
     <geometry>
-      <mesh filename="package://openarm_grip_description/meshes/right_jaw_1.stl" scale="0.001 0.001 0.001"/>
+      <mesh filename="package://openarm_description/meshes/right_jaw_1.stl" scale="0.001 0.001 0.001"/>
     </geometry>
   </collision>

File: openarm_moveit_config/config/openarm_grip.urdf.xacro (robot description, xacro)
@@ -1,9 +1,9 @@
 <?xml version="1.0"?>
-<robot xmlns:xacro="http://www.ros.org/wiki/xacro" name="openarm_grip">
+<robot xmlns:xacro="http://www.ros.org/wiki/xacro" name="openarm">
     <xacro:arg name="initial_positions_file" default="initial_positions.yaml" />
-    <!-- Import openarm_grip urdf file -->
-    <xacro:include filename="$(find openarm_grip_description)/urdf/openarm_grip.urdf" />
+    <!-- Import openarm urdf file -->
+    <xacro:include filename="$(find openarm_description)/urdf/openarm.urdf" />
     <!-- Import control_xacro -->
-    <xacro:include filename="openarm_grip.ros2_control.xacro" />
-    <xacro:openarm_grip_ros2_control name="FakeSystem" initial_positions_file="$(arg initial_positions_file)"/>
+    <xacro:include filename="openarm.ros2_control.xacro" />
+    <xacro:openarm_ros2_control name="FakeSystem" initial_positions_file="$(arg initial_positions_file)"/>
 </robot>
