Commit message: Restore joints to main state

File: openarm_description/urdf/openarm.urdf (robot description, URDF)
Before this commit: robot openarm, 11 links, 9 joints
Links:
- removed link dummy
- added link world
Joints:
- removed joint dummy_joint
- added joint slider_right: type prismatic, parent grip_attach_1, child right_jaw_1, origin xyz=0.0775 -0.121655 0.012086 rpy=0 0 0, axis 1.0 -0.0 0.0, limit lower=-0.0455 upper=0.0 effort=100 velocity=1.0, mimic joint=slider_left
- added joint world_joint: type fixed, parent world, child base_link, origin xyz=0.0 0.0 0.0 rpy=0.0 0.0 0.0
- joint rev7: limit (none) -> lower=-1.5 upper=1.5 effort=100 velocity=1.0; type continuous -> revolute
- joint slider_left: axis 1.0 -0.0 0.0 -> -1.0 0.0 -0.0; child right_jaw_1 -> left_jaw_1; origin xyz=0.0775 -0.121655 0.012086 rpy=0 0 0 -> xyz=-0.0775 -0.121655 0.012086 rpy=0 0 0

File: openarm_description/urdf/openarm.xacro (robot description, xacro)
@@ -1,10 +1,10 @@
 <?xml version="1.0" ?>
 <robot name="openarm" xmlns:xacro="http://www.ros.org/wiki/xacro">
-<xacro:include filename="$(find openarm_description)/urdf/materials.xacro" />
-<xacro:include filename="$(find openarm_description)/urdf/openarm.trans" />
-<xacro:include filename="$(find openarm_description)/urdf/openarm.gazebo" />
-<link name="dummy"/>
-<joint name="dummy_joint" type="fixed">
-  <parent link="dummy"/>
+<xacro:include filename="materials.xacro" />
+<xacro:include filename="openarm.trans" />
+<xacro:include filename="openarm.gazebo" />
+<link name="world"/>
+<joint name="world_joint" type="fixed">
+  <parent link="world"/>
   <child link="base_link"/>
   <origin xyz="0.0 0.0 0.0" rpy="0.0 0.0 0.0"/>
@@ -216,4 +216,5 @@
   <axis xyz="0.0 0.0 1.0"/>
   <limit upper="2.356194" lower="-2.356194" effort="100" velocity="1.0" acceleration="0.5"/>
+  <dynamics damping="1.0" friction="1.0"/>
 </joint>
 <joint name="rev2" type="revolute">
@@ -223,4 +224,5 @@
   <axis xyz="-1.0 -0.0 0.0"/>
   <limit upper="0.0" lower="-3.054326" effort="100" velocity="1.0" acceleration="0.5"/>
+  <dynamics damping="1.0" friction="1.0"/>
 </joint>
 <joint name="rev3" type="revolute">
@@ -230,4 +232,5 @@
   <axis xyz="-0.0 0.986291 0.165017"/>
   <limit upper="2.094395" lower="-2.094395" effort="100" velocity="1.0" acceleration="0.5"/>
+  <dynamics damping="1.0" friction="1.0"/>
 </joint>
 <joint name="rev4" type="revolute">
@@ -237,4 +240,5 @@
   <axis xyz="1.0 0.0 0.0"/>
   <limit upper="0.0" lower="-3.141593" effort="100" velocity="1.0" acceleration="0.5"/>
+  <dynamics damping="1.0" friction="1.0"/>
 </joint>
 <joint name="rev5" type="revolute">
@@ -244,4 +248,5 @@
   <axis xyz="0.0 -0.980588 0.196078"/>
   <limit upper="2.094395" lower="-2.094395" effort="100" velocity="1.0" acceleration="0.5"/>
+  <dynamics damping="1.0" friction="1.0"/>
 </joint>
 <joint name="rev6" type="revolute">
@@ -251,10 +256,13 @@
   <axis xyz="-1.0 0.0 -0.0"/>
   <limit upper="1.570796" lower="-1.570796" effort="100" velocity="1.0" acceleration="0.5"/>
-</joint>
-<joint name="rev7" type="continuous">
+  <dynamics damping="1.0" friction="1.0"/>
+</joint>
+<joint name="rev7" type="revolute">
   <origin xyz="-0.0355 0.00303 0.01515" rpy="0 0 0"/>
   <parent link="J7_v1_1"/>
   <child link="grip_attach_1"/>
   <axis xyz="0.0 0.196078 0.980588"/>
+  <limit upper="0.5" lower="-0.5" effort="100" velocity="1.0" acceleration="0.5"/>
+  <dynamics damping="1.0" friction="1.0"/>
 </joint>
 <joint name="slider_left" type="prismatic">
@@ -264,6 +272,7 @@
   <axis xyz="-1.0 0.0 -0.0"/>
   <limit upper="0.0" lower="-0.0455" effort="100" velocity="1.0" acceleration="0.5"/>
-</joint>
-<joint name="slider_left" type="prismatic">
+  <dynamics damping="1.0" friction="1.0"/>
+</joint>
+<joint name="slider_right" type="prismatic">
   <origin xyz="0.0775 -0.121655 0.012086" rpy="0 0 0"/>
   <parent link="grip_attach_1"/>
@@ -271,4 +280,6 @@
   <axis xyz="1.0 -0.0 0.0"/>
   <limit upper="0.0" lower="-0.0455" effort="100" velocity="1.0" acceleration="0.5"/>
+  <dynamics damping="1.0" friction="1.0"/>
+  <mimic joint="slider_left"/>
 </joint>
 </robot>
