Commit message: Tune motor1 KP and reset right arm rev2 params to proper arm configuration

File: openarm_description/urdf/openarm.xacro (robot description, xacro)
@@ -232,6 +232,6 @@
             <child link="${prefix}link3"/>
             <origin rpy="-1.5707963267948968 ${pi/2 if zero_pos=='up' else 0.0} 0.0" xyz="0.0 -0.02975 0.04475"/>
-            <axis xyz="0 0 ${reflect * -1}"/>
-            <limit effort="0.0" lower="${-pi/2.0 if zero_pos=='up' else -pi + rotate}" upper="${pi/2 if zero_pos=='up' else 0 + rotate}" velocity="0.0"/>
+            <axis xyz="0 0 1"/>
+            <limit effort="0.0" lower="${-pi/2.0 if zero_pos=='up' else 0.0}" upper="${pi/2 if zero_pos=='up' else pi}" velocity="0.0"/>
         </joint>
         <joint name="${prefix}rev3" type="revolute">
